File: KiCAD/KZ80-TMS9918A.kicad_pcb (KiCad board)
At the start: 2 copper layers, 100 x 75 mm, 38 parts, among them J1 Conn_Coaxial, J2 SBC8080 BUS, J3 EXT_JP, J4 AD_JP, J5 AD_JP, Q1 2SC1815, U1 74HCT04, U2 74HC139, U3 74HC32, U4 TMS9918A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

Commit message: RCAコネクタフットプリント作成。出力回路見直し
Parts:
- added C14: 0.1u, Capacitor_THT:C_Disc_D3.0mm_W1.6mm_P2.50mm, F.Cu at (127.0, 107.5)
- added C15: 470u, Capacitor_THT:CP_Radial_D8.0mm_P3.50mm, F.Cu at (138.0, 106.5)
- added R4: 75, Resistor_THT:R_Axial_DIN0207_L6.3mm_D2.5mm_P10.16mm_Horizontal, F.Cu at (141.0, 122.5)
- added R5: 10k, Resistor_THT:R_Axial_DIN0207_L6.3mm_D2.5mm_P10.16mm_Horizontal, F.Cu at (136.5, 112.5)
- C3: value 0.1U -> 10u; footprint Capacitor_THT:C_Disc_D3.0mm_W1.6mm_P2.50mm -> Capacitor_THT:CP_Radial_D5.0mm_P2.50mm
- J1: footprint Connector_Coaxial:SMA_Molex_73251-1153_EdgeMount_Horizontal -> RCACon:RCAConAE
- R1: value 75 -> 300
- moved C4 8.50 mm to (113.5, 94.5)
- moved C3 4.30 mm to (139.0, 97.5)
- moved J1 3.54 mm to (128.0, 117.5), turned to 180 degrees
Connections:
- J4 pad 4: Net-(J4-Pad4) -> Net-(J4-Pad2)
- J4 pad 6: Net-(J4-Pad5) -> Net-(J4-Pad2)
- J4 pad 7: Net-(J4-Pad5) -> Net-(J4-Pad7)
- J4 pad 8: Net-(J4-Pad5) -> Net-(J4-Pad2)
- J5 pad 4: Net-(J5-Pad4) -> Net-(J5-Pad2)
- J5 pad 6: Net-(J5-Pad5) -> Net-(J5-Pad2)
- J5 pad 7: Net-(J5-Pad5) -> Net-(J5-Pad7)
- J5 pad 8: Net-(J5-Pad5) -> Net-(J5-Pad2)
- Q1 pad 1: Net-(J1-Pad1) -> Net-(C15-Pad1)
- R1 pad 1: Net-(J1-Pad1) -> Net-(C15-Pad1)
- U2 pad 10: Net-(J4-Pad3) -> Net-(J4-Pad5)
- U2 pad 11: Net-(J4-Pad2) -> Net-(J4-Pad3)
- U2 pad 15: Net-(J5-Pad5) -> Net-(J5-Pad2)
- U2 pad 5: Net-(J5-Pad2) -> Net-(J5-Pad3)
- U2 pad 6: Net-(J5-Pad3) -> Net-(J5-Pad5)
- U2 pad 7: Net-(J5-Pad4) -> Net-(J5-Pad7)
- U2 pad 9: Net-(J4-Pad4) -> Net-(J4-Pad7)
- U3 pad 1: Net-(J4-Pad5) -> Net-(J4-Pad2)
- U3 pad 4: Net-(J4-Pad5) -> Net-(J4-Pad2)
- U4 pad 17: /D7 -> /D0
- U4 pad 18: /D6 -> /D1
- U4 pad 19: /D5 -> /D2
- U4 pad 20: /D4 -> /D3
- U4 pad 21: /D3 -> /D4
- U4 pad 22: /D2 -> /D5
- U4 pad 23: /D1 -> /D6
- U4 pad 24: /D0 -> /D7
Routing:
- net Net-(J5-Pad2): track 17.3 -> 55.0 mm
- net /D1: track 57.7 -> 93.7 mm
- net /D2: track 57.6 -> 90.9 mm
- net GND: track 380.8 -> 411.9 mm, vias 1 -> 0
- net Net-(J5-Pad7): track 0.00 -> 27.3 mm
- net Net-(C15-Pad1): track 0.00 -> 25.5 mm
- net /D3: track 63.8 -> 88.2 mm
- net Net-(J4-Pad2): track 16.0 -> 39.5 mm
- net /D0: track 52.6 -> 75.0 mm
- net /~CAS: track 144.3 -> 122.1 mm
- net Net-(J5-Pad5): track 43.6 -> 22.2 mm
- net /AD2: track 94.1 -> 73.9 mm, vias 1 -> 0
- net Net-(J4-Pad7): track 0.00 -> 19.6 mm
- net /AD5: track 137.9 -> 118.4 mm
- net /RES: track 48.6 -> 29.9 mm, vias 0 -> 1
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- added copper zone on B.Cu, net GND
- added copper zone on F.Cu, net GND
Other:
- board text added: "00"
- board text added: "08"
- board text added: "10"
- board text added: "18"
- board text added: "20"
- board text added: "40"
- board text added: "60"
- board text added: "80"
- board text added: "CLK"
- board text added: "CPUCLK"
- board text added: "EXT"
- board text added: "GND"
- board text added: "GRM"
- board text added: "INT"
